File: hardware/src/Door_Client.brd (EAGLE design)
At the start: 84.1 x 69.8 mm, 41 parts, among them IC1 L272M, IC2 MAX3468EPA, IC3 MC78M05ABT, IC4 4050N, J1 HEAD15-NOSS, J2 HEAD15-NOSS-1, Q1 TIP42C, X1 22-23-2021

Commit message: Re-organize and update board layout files
Parts:
- removed PROG1: (no value), pinhead:1X03
- removed READER: (no value), pinhead:1X09
- added DOORBELL, LCD: (no value), pinhead:1X03
- added JP1: (no value), pinhead:1X08
- moved R16 57.2 mm to (21.6, 57.1), turned to 180 degrees
- moved LED2 48.4 mm to (27.9, 54.6), turned to 0 degrees
- moved LATCH_OUTPUT 12.7 mm to (76.2, 50.2)
- moved DOOR_CLOSE 10.2 mm to (76.2, 37.5)
- moved EXIT_BUTTON 7.62 mm to (76.2, 24.8)
- moved D1 7.62 mm to (69.2, 48.3)
- moved AUDIO 6.84 mm to (17.1, 67.3)
- moved IC3 6.35 mm to (65.4, 61.6)
- moved PWR 6.35 mm to (65.4, 69.2)
- moved Q1 5.24 mm to (66.7, 44.5)
- moved C2 5.08 mm to (31.8, 64.1)
- moved IC1 5.08 mm to (40.6, 60.3)
- moved T3 5.08 mm to (57.1, 44.5)
- moved PROG 5.08 mm to (31.8, 30.5)
- moved R3 5.08 mm to (64.1, 27.9)
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Connections:
- net +5V: now also DOORBELL.3, LCD.3; no longer PROG1.3
- net 3V3: now also JP1.1; no longer READER.1
- net A3: now also DOORBELL.1
- net COM: now also DOORBELL.2, JP1.3, LCD.2; no longer PROG1.2, READER.8
- net D12/MISO: now also JP1.5; no longer READER.3
- net D4: now also LCD.1; no longer PROG1.1
- net N$19: now also JP1.7; no longer READER.2
- net N$20: now also JP1.6; no longer READER.4
- net N$21: now also JP1.8; no longer READER.5
- net N$3: now also JP1.2; no longer READER.6
Routing:
- net COM: track 536.5 -> 611.6 mm
- net A3: track 0.00 -> 34.2 mm
- net N$3: track 37.7 -> 13.0 mm
- net N$19: track 20.1 -> 40.0 mm
- net +5V: track 173.5 -> 188.8 mm
- net D3: track 59.3 -> 51.6 mm
- net D4: track 61.1 -> 53.5 mm
- net N$11: track 23.2 -> 27.0 mm
- net D12/MISO: track 29.5 -> 32.6 mm
- net N$14: track 8.50 -> 10.5 mm
- net N$12: track 4.49 -> 2.54 mm
- net N$21: track 22.3 -> 20.6 mm
- net N$10: track 9.26 -> 10.8 mm
- net N$16: track 8.01 -> 9.44 mm
- net D2: track 35.4 -> 36.7 mm
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Other:
- board size 84.1 x 69.8 mm -> 84.1 x 77.5 mm
- board text added: "3.3v"
- board text added: "5v"
- board text added: "GND"
- board text added: "RX"
