File: hardware/src/Mini_Door_Client.brd (EAGLE design)
At the start: 11 x 38.9 mm, 6 parts

Commit message: New client board V0.1
Changed lines of the file:
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@@
 <?xml version="1.0" encoding="utf-8"?>
 <!DOCTYPE eagle SYSTEM "eagle.dtd">
-<eagle version="7.5.0">
+<eagle version="7.7.0">
 <drawing>
 <settings>
@@
 <board>
 <plain>
-<wire x1="-0.396240625" y1="-0.396240625" x2="10.556240625" y2="-0.396240625" width="0.79248125" layer="46"/>
-<wire x1="10.556240625" y1="-0.396240625" x2="10.556240625" y2="38.496240625" width="0.79248125" layer="46"/>
-<wire x1="10.556240625" y1="38.496240625" x2="-0.396240625" y2="38.496240625" width="0.79248125" layer="46"/>
-<wire x1="-0.396240625" y1="38.496240625" x2="-0.396240625" y2="-0.396240625" width="0.79248125" layer="46"/>
+<wire x1="-0.396240625" y1="-0.396240625" x2="10.556240625" y2="-0.396240625" width="0.254" layer="20"/>
+<wire x1="10.556240625" y1="-0.396240625" x2="10.556240625" y2="38.496240625" width="0.254" layer="20"/>
+<wire x1="10.556240625" y1="38.496240625" x2="-0.396240625" y2="38.496240625" width="0.254" layer="20"/>
+<wire x1="-0.396240625" y1="38.496240625" x2="-0.396240625" y2="-0.396240625" width="0.254" layer="20"/>
 </plain>
 <attributes>
